File: 02/pcb-v4/pcb-2.kicad_sch (KiCad schematic)
At the start: 44 parts, among them U1 Arduino_Pro_Micro, U2 TRRS

Commit message: fix: reversible footprints — schematic sync, TRRS, DRC flags
- Updated pcb-2.kicad_sch: all 21 diodes, 21 switches, and TRRS now
  reference Library:* footprints so KiCad won't revert them on re-open
- Added Library:TRRS_PJ-320A_reversible with F.SilkS + B.SilkS body
  outline and F.CrtYd + B.CrtYd courtyard (TH pads already *.Cu)
- Re-ran diode swap (KiCad had reverted to Scotto library versions)
- Set duplicate_pad_numbers_are_jumpers yes on all 42 reversible
  footprints (switches + diodes) — fixes the DRC duplicate-pad errors

Co-Authored-By: Claude Sonnet 4.6 <noreply@anthropic.com>
Parts:
- D1, D10, D11, D12, D13, D14, D15, D16, D17, D18, D19, D2, D20, D21, D3, D4, D5, D6, D7, D8, D9: footprint Scotto Components:Diode_SOD-123 -> Library:Diode_SOD-123_reversible
- S1, S10, S11, S12, S13, S14, S15, S16, S17, S18, S19, S2, S20, S21, S3, S4, S5, S6, S7, S8, S9: footprint PCM_Switch_Keyboard_Hotswap_Kailh:SW_Hotswap_Kailh_Choc_V1 -> Library:Kailh_socket_PG1350_reversible
- U2: footprint ScottoKeebs_Components:TRRS_PJ-320A -> Library:TRRS_PJ-320A_reversible
Changed lines of the file:
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@@
 			)
 		)
-		(property "Footprint" "PCM_Switch_Keyboard_Hotswap_Kailh:SW_Hotswap_Kailh_Choc_V1"
+		(property "Footprint" "Library:Kailh_socket_PG1350_reversible"
 			(at 143.51 59.69 0)
 			(hide yes)
@@
 			)
 		)
-		(property "Footprint" "Scotto Components:Diode_SOD-123"
+		(property "Footprint" "Library:Diode_SOD-123_reversible"
 			(at 90.17 66.04 0)
 			(hide yes)
@@
 			)
 		)
-		(property "Footprint" "PCM_Switch_Keyboard_Hotswap_Kailh:SW_Hotswap_Kailh_Choc_V1"
+		(property "Footprint" "Library:Kailh_socket_PG1350_reversible"
 			(at 101.6 81.28 0)
 			(hide yes)
@@
 			)
 		)
-		(property "Footprint" "Scotto Components:Diode_SOD-123"
+		(property "Footprint" "Library:Diode_SOD-123_reversible"
 			(at 132.08 109.22 0)
 			(hide yes)
@@
 			)
 		)
-		(property "Footprint" "Scotto Components:Diode_SOD-123"
+		(property "Footprint" "Library:Diode_SOD-123_reversible"
 			(at 118.11 109.22 0)
 			(hide yes)
@@
 			)
 		)
-		(property "Footprint" "Scotto Components:Diode_SOD-123"
+		(property "Footprint" "Library:Diode_SOD-123_reversible"
 			(at 118.11 87.63 0)
 			(hide yes)
@@
 			)
 		)
-		(property "Footprint" "PCM_Switch_Keyboard_Hotswap_Kailh:SW_Hotswap_Kailh_Choc_V1"
+		(property "Footprint" "Library:Kailh_socket_PG1350_reversible"
 			(at 87.63 59.69 0)
 			(hide yes)
@@
 			)
 		)
-		(property "Footprint" "PCM_Switch_Keyboard_Hotswap_Kailh:SW_Hotswap_Kailh_Choc_V1"
+		(property "Footprint" "Library:Kailh_socket_PG1350_reversible"
 			(at 129.54 124.46 0)
 			(hide yes)
@@
 			)
 		)
-		(property "Footprint" "PCM_Switch_Keyboard_Hotswap_Kailh:SW_Hotswap_Kailh_Choc_V1"
+		(property "Footprint" "Library:Kailh_socket_PG1350_reversible"
 			(at 143.51 124.46 0)
 			(hide yes)
@@
 			)
 		)
-		(property "Footprint" "Scotto Components:Diode_SOD-123"
+		(property "Footprint" "Library:Diode_SOD-123_reversible"
 			(at 160.02 130.81 0)
 			(hide yes)
@@
 			)
 		)
-		(property "Footprint" "Scotto Components:Diode_SOD-123"
+		(property "Footprint" "Library:Diode_SOD-123_reversible"
 			(at 90.17 87.63 0)
 			(hide yes)
@@
 			)
 		)
-		(property "Footprint" "PCM_Switch_Keyboard_Hotswap_Kailh:SW_Hotswap_Kailh_Choc_V1"
+		(property "Footprint" "Library:Kailh_socket_PG1350_reversible"
 			(at 143.51 81.28 0)
 			(hide yes)
@@
 			)
 		)
-		(property "Footprint" "PCM_Switch_Keyboard_Hotswap_Kailh:SW_Hotswap_Kailh_Choc_V1"
+		(property "Footprint" "Library:Kailh_socket_PG1350_reversible"
 			(at 87.63 81.28 0)
 			(hide yes)
@@
 			)
 		)
-		(property "Footprint" "Scotto Components:Diode_SOD-123"
+		(property "Footprint" "Library:Diode_SOD-123_reversible"
 			(at 146.05 87.63 0)
 			(hide yes)
@@
 			)
 		)
-		(property "Footprint" "Scotto Components:Diode_SOD-123"
+		(property "Footprint" "Library:Diode_SOD-123_reversible"
 			(at 160.02 109.22 0)
 			(hide yes)
@@
 			)
 		)
-		(property "Footprint" "Scotto Components:Diode_SOD-123"
+		(property "Footprint" "Library:Diode_SOD-123_reversible"
 			(at 146.05 130.81 0)
 			(hide yes)
@@
 			)
 		)
-		(property "Footprint" "Scotto Components:Diode_SOD-123"
+		(property "Footprint" "Library:Diode_SOD-123_reversible"
 			(at 160.02 87.63 0)
 			(hide yes)
@@
 			)
 		)
-		(property "Footprint" "PCM_Switch_Keyboard_Hotswap_Kailh:SW_Hotswap_Kailh_Choc_V1"
+		(property "Footprint" "Library:Kailh_socket_PG1350_reversible"
 			(at 115.57 102.87 0)
 			(hide yes)
@@
 			)
 		)
-		(property "Footprint" "PCM_Switch_Keyboard_Hotswap_Kailh:SW_Hotswap_Kailh_Choc_V1"
+		(property "Footprint" "Library:Kailh_socket_PG1350_reversible"
 			(at 157.48 81.28 0)
 			(hide yes)
@@
 			)
 		)
-		(property "Footprint" "Scotto Components:Diode_SOD-123"
+		(property "Footprint" "Library:Diode_SOD-123_reversible"
 			(at 104.14 66.04 0)
 			(hide yes)
@@
 			)
 		)
-		(property "Footprint" "Scotto Components:Diode_SOD-123"
+		(property "Footprint" "Library:Diode_SOD-123_reversible"
 			(at 146.05 66.04 0)
 			(hide yes)
@@
 			)
 		)
-		(property "Footprint" "PCM_Switch_Keyboard_Hotswap_Kailh:SW_Hotswap_Kailh_Choc_V1"
+		(property "Footprint" "Library:Kailh_socket_PG1350_reversible"
 			(at 115.57 81.28 0)
 			(hide yes)
@@
 			)
 		)
-		(property "Footprint" "Scotto Components:Diode_SOD-123"
+		(property "Footprint" "Library:Diode_SOD-123_reversible"
 			(at 160.02 66.04 0)
 			(hide yes)
@@
 			)
 		)
-		(property "Footprint" "PCM_Switch_Keyboard_Hotswap_Kailh:SW_Hotswap_Kailh_Choc_V1"
+		(property "Footprint" "Library:Kailh_socket_PG1350_reversible"
 			(at 115.57 59.69 0)
 			(hide yes)
@@
 			)
 		)
-		(property "Footprint" "Scotto Components:Diode_SOD-123"
+		(property "Footprint" "Library:Diode_SOD-123_reversible"
 			(at 104.14 109.22 0)
 			(hide yes)
@@
 			)
 		)
-		(property "Footprint" "PCM_Switch_Keyboard_Hotswap_Kailh:SW_Hotswap_Kailh_Choc_V1"
+		(property "Footprint" "Library:Kailh_socket_PG1350_reversible"
 			(at 157.48 124.46 0)
 			(hide yes)
@@
 			)
 		)
-		(property "Footprint" "Scotto Components:Diode_SOD-123"
+		(property "Footprint" "Library:Diode_SOD-123_reversible"
 			(at 104.14 87.63 0)
 			(hide yes)
@@
 			)
 		)
-		(property "Footprint" "Scotto Components:Diode_SOD-123"
+		(property "Footprint" "Library:Diode_SOD-123_reversible"
 			(at 146.05 109.22 0)
 			(hide yes)
@@
 			)
 		)
-		(property "Footprint" "PCM_Switch_Keyboard_Hotswap_Kailh:SW_Hotswap_Kailh_Choc_V1"
+		(property "Footprint" "Library:Kailh_socket_PG1350_reversible"
 			(at 143.51 102.87 0)
 			(hide yes)
@@
 			)
 		)
-		(property "Footprint" "Scotto Components:Diode_SOD-123"
+		(property "Footprint" "Library:Diode_SOD-123_reversible"
 			(at 118.11 66.04 0)
 			(hide yes)
@@
 			)
 		)
-		(property "Footprint" "PCM_Switch_Keyboard_Hotswap_Kailh:SW_Hotswap_Kailh_Choc_V1"
+		(property "Footprint" "Library:Kailh_socket_PG1350_reversible"
 			(at 101.6 59.69 0)
 			(hide yes)
@@
 			)
 		)
-		(property "Footprint" "PCM_Switch_Keyboard_Hotswap_Kailh:SW_Hotswap_Kailh_Choc_V1"
+		(property "Footprint" "Library:Kailh_socket_PG1350_reversible"
 			(at 129.54 59.69 0)
 			(hide yes)
@@
 			)
 		)
-		(property "Footprint" "Scotto Components:Diode_SOD-123"
+		(property "Footprint" "Library:Diode_SOD-123_reversible"
 			(at 132.08 130.81 0)
 			(hide yes)
@@
 			)
 		)
-		(property "Footprint" "Scotto Components:Diode_SOD-123"
+		(property "Footprint" "Library:Diode_SOD-123_reversible"
 			(at 132.08 66.04 0)
 			(hide yes)
@@
 			)
 		)
-		(property "Footprint" "PCM_Switch_Keyboard_Hotswap_Kailh:SW_Hotswap_Kailh_Choc_V1"
+		(property "Footprint" "Library:Kailh_socket_PG1350_reversible"
 			(at 101.6 102.87 0)
 			(hide yes)
@@
 			)
 		)
-		(property "Footprint" "Scotto Components:Diode_SOD-123"
+		(property "Footprint" "Library:Diode_SOD-123_reversible"
 			(at 132.08 87.63 0)
 			(hide yes)
@@
 			)
 		)
-		(property "Footprint" "ScottoKeebs_Components:TRRS_PJ-320A"
+		(property "Footprint" "Library:TRRS_PJ-320A_reversible"
 			(at 229.87 147.32 0)
 			(hide yes)
@@
 			)
 		)
-		(property "Footprint" "PCM_Switch_Keyboard_Hotswap_Kailh:SW_Hotswap_Kailh_Choc_V1"
+		(property "Footprint" "Library:Kailh_socket_PG1350_reversible"
 			(at 87.63 102.87 0)
 			(hide yes)
@@
 			)
 		)
-		(property "Footprint" "PCM_Switch_Keyboard_Hotswap_Kailh:SW_Hotswap_Kailh_Choc_V1"
+		(property "Footprint" "Library:Kailh_socket_PG1350_reversible"
 			(at 129.54 102.87 0)
 			(hide yes)
@@
 			)
 		)
-		(property "Footprint" "PCM_Switch_Keyboard_Hotswap_Kailh:SW_Hotswap_Kailh_Choc_V1"
+		(property "Footprint" "Library:Kailh_socket_PG1350_reversible"
 			(at 157.48 102.87 0)
 			(hide yes)
@@
 			)
 		)
-		(property "Footprint" "PCM_Switch_Keyboard_Hotswap_Kailh:SW_Hotswap_Kailh_Choc_V1"
+		(property "Footprint" "Library:Kailh_socket_PG1350_reversible"
 			(at 129.54 81.28 0)
 			(hide yes)
@@
 			)
 		)
-		(property "Footprint" "Scotto Components:Diode_SOD-123"
+		(property "Footprint" "Library:Diode_SOD-123_reversible"
 			(at 90.17 109.22 0)
 			(hide yes)
@@
 			)
 		)
-		(property "Footprint" "PCM_Switch_Keyboard_Hotswap_Kailh:SW_Hotswap_Kailh_Choc_V1"
+		(property "Footprint" "Library:Kailh_socket_PG1350_reversible"
 			(at 157.48 59.69 0)
 			(hide yes)
