File: 02/pcb-v4/pcb-2.kicad_pcb (KiCad board)
At the start: 2 copper layers, 146.9 x 86 mm, 44 parts, among them U1 Arduino_Pro_Micro, U2 TRRS

Commit message: feat: working on 02
Routing:
- net Column 1: track 419.4 -> 188.9 mm, vias 7 -> 18
- net Column 2: track 402.4 -> 182.5 mm, vias 13 -> 21
- net Column 3: track 337.1 -> 182.4 mm, vias 13 -> 25
- net Column 6: track 218.6 -> 107.8 mm, vias 11 -> 19
- net Column 4: track 276.8 -> 166.3 mm, vias 13 -> 22
- net Column 5: track 245.5 -> 142.5 mm, vias 12 -> 23
- net Row 1: track 162.6 -> 136.7 mm, vias 0 -> 16
- net Net-(D1-A): track 2.57 -> 25.4 mm, vias 0 -> 2
- net Net-(D10-A): track 7.34 -> 28.7 mm, vias 0 -> 5
- net Net-(D12-A): track 4.96 -> 26.3 mm, vias 0 -> 5
- net Net-(D11-A): track 4.96 -> 25.5 mm, vias 0 -> 2
- net Net-(D16-A): track 9.72 -> 30.2 mm, vias 0 -> 9
- net Net-(D15-A): track 4.96 -> 25.3 mm, vias 0 -> 4
- net Net-(D5-A): track 4.96 -> 24.8 mm, vias 0 -> 3
- net Net-(D17-A): track 4.96 -> 24.8 mm, vias 0 -> 2
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